File: fx2la_interface.kicad_pcb (KiCad board)
At the start: 2 copper layers, 19 x 18 mm, 14 parts, among them J1 Cortex-Debug, J2 Cortex-Debug, J3 Conn_02x05_Counter_Clockwise

Commit message: Separate connectors more
Parts:
- added TP3: TestPoint, connectors:pad_1.5x2.0mm, F.Cu at (138.0, 88.5)
- added kibuzzard-63A316D6: G***, kibuzzard-63A316D6, F.Cu at (138.0, 84.8)
- moved J1 3.25 mm to (148.0, 69.8)
- moved J2 3.25 mm to (148.0, 86.2)
- moved TP2 3.00 mm to (142.0, 88.5)
- moved kibuzzard-639836FB 3.00 mm to (142.0, 84.8)
Routing:
- net /RST: track 29.1 -> 37.1 mm
- net /SWDIO: track 30.1 -> 37.9 mm
- net /TDI: track 30.9 -> 38.7 mm
- net /SWCLK: track 31.8 -> 39.7 mm
- net /KEY: track 25.8 -> 32.4 mm, vias 2 -> 3
- net /VREF: track 16.7 -> 23.2 mm
- net /GND_DETECT: track 25.4 -> 29.5 mm
- net /SWO: track 42.7 -> 45.0 mm
- net GND: vias 4 -> 28
- added copper zone on F.Cu, net GND
Other:
- board size 19 x 18 mm -> 19 x 24 mm
