File: fx2la_interface.kicad_sch (KiCad schematic)
At the start: 5 parts, among them J1 Cortex-Debug, J2 Cortex-Debug, J3 Conn_02x05_Counter_Clockwise

Commit message: Separate connectors more
Parts:
- added TP3: TestPoint, connectors:pad_1.5x2.0mm, symbol Connector:TestPoint
Connections:
- net GND: now also TP3.1
Changed lines of the file:
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@@
     (pin "9")
+  )
+  (symbol (lib_id "power:GND") (at 67.31 73.66 0) (unit 1)
+    (in_bom yes) (on_board yes) (fields_autoplaced)
+    (property "Reference" "#PWR0101" (id 0) (at 67.31 80.01 0)
+      (effects (font (size 1.27 1.27)) hide)
+    )
+    (property "Value" "GND" (id 1) (at 67.31 78.74 0)
+      (effects (font (size 1.27 1.27)) hide)
+    )
+    (property "Footprint" "" (id 2) (at 67.31 73.66 0)
+      (effects (font (size 1.27 1.27)) hide)
+    )
+    (property "Datasheet" "" (id 3) (at 67.31 73.66 0)
+      (effects (font (size 1.27 1.27)) hide)
+    )
+    (pin "1")
   )
   (symbol (lib_id "power:GND") (at 71.12 104.14 270) (unit 1)
@@
     (pin "9")
   )
+  (symbol (lib_id "Connector:TestPoint") (at 67.31 73.66 0) (unit 1)
+    (in_bom no) (on_board yes) (fields_autoplaced)
+    (property "Reference" "TP3" (id 0) (at 69.85 69.0879 0)
+      (effects (font (size 1.27 1.27)) (justify left))
+    )
+    (property "Value" "TestPoint" (id 1) (at 69.85 71.6279 0)
+      (effects (font (size 1.27 1.27)) (justify left))
+    )
+    (property "Footprint" "connectors:pad_1.5x2.0mm" (id 2) (at 72.39 73.66 0)
+      (effects (font (size 1.27 1.27)) hide)
+    )
+    (property "Datasheet" "~" (id 3) (at 72.39 73.66 0)
+      (effects (font (size 1.27 1.27)) hide)
+    )
+    (pin "1")
+  )
   (symbol (lib_id "power:GND") (at 119.38 104.14 270) (unit 1)
     (in_bom yes) (on_board yes) (fields_autoplaced)
@@
       (reference "#PWR05") (unit 1) (value "GND") (footprint "")
     )
+    (path "/6d14666d-1036-4553-b5c1-2828f47d1cc7"
+      (reference "#PWR0101") (unit 1) (value "GND") (footprint "")
+    )
     (path "/9e4e9e48-5ab8-4abf-a1b7-35d11011e2b2"
       (reference "J1") (unit 1) (value "Cortex-Debug") (footprint "connectors:PinHeader_2x05_FTSH-105-01-L-DV-K")
@@
       (reference "TP2") (unit 1) (value "TestPoint") (footprint "connectors:pad_1.5x2.0mm")
     )
+    (path "/aa24e64e-415d-4552-838d-99aec595dcb5"
+      (reference "TP3") (unit 1) (value "TestPoint") (footprint "connectors:pad_1.5x2.0mm")
+    )
   )
